File: iot node/iot node.kicad_sch (KiCad schematic)
At the start: 43 parts, among them J1 Conn_01x04_Female, J2 Conn_01x06_Female, SW1 SW_Push, SW2 SW_Push, SW3 SW_Push, U1 ESP32-C3-WROOM-02, U2 NCP1117-3.3_SOT223, U3 EKMB1305112K, U4 BME680, X1 DG3XX-02-5.0

Commit message: voltage suply adapt
Parts:
- removed U2: NCP1117-3.3_SOT223, Package_TO_SOT_SMD:SOT-223-3_TabPin2, symbol Regulator_Linear:NCP1117-3.3_SOT223
- added R5: 4.7k, Resistor_SMD:R_0805_2012Metric_Pad1.20x1.40mm_HandSolder, symbol Device:R
- added U2: LP2989IMX-3.3/NOPB, LP2989IMX-3:SOIC127P600X175-8N, symbol LP2989IMX-3.3_NOPB:LP2989IMX-3.3/NOPB
- C4: value 10u -> 2.2u
- C5: value 10u -> 4.7u
- renumbered R5 to R6, R6 to R7, R7 to R8, R8 to R9, TP7 to TP6, TP6 to TP7
Connections:
- net + suply : now also U2.4 (INPUT)
- net 3.3: now also R5.1, U2.5 (OUTPUT)
- net GND: now also U2.3 (GND)
- new net: R5.2, U2.7 (~{ERROR})
- no-connect marks 5 -> 8
Other:
- moved on the sheet: C4, C5, J2, R3, R4, TP4, TP5, TP7, X1A, X1B

Commit message: pcb
Parts:
- removed TP12: TestPoint, Connector_Pin:Pin_D0.7mm_L6.5mm_W1.8mm_FlatFork, symbol Connector:TestPoint
- R9: value 10k -> 1meg
Changed lines of the file:
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@@
   (junction (at 33.02 173.99) (diameter 0) (color 0 0 0 0)
-  )
-  (junction (at 227.33 99.06) (diameter 0) (color 0 0 0 0)
   )
   (junction (at 246.38 132.08) (diameter 0) (color 0 0 0 0)
@@
     (stroke (width 0) (type default) (color 0 0 0 0))
   )
-  (wire (pts (xy 226.06 99.06) (xy 227.33 99.06))
+  (wire (pts (xy 226.06 99.06) (xy 234.95 99.06))
     (stroke (width 0) (type default) (color 0 0 0 0))
   )
@@
   )
   (wire (pts (xy 33.02 173.99) (xy 41.91 173.99))
-    (stroke (width 0) (type default) (color 0 0 0 0))
-  )
-  (wire (pts (xy 227.33 99.06) (xy 234.95 99.06))
     (stroke (width 0) (type default) (color 0 0 0 0))
   )
@@
       (effects (font (size 1.27 1.27)) (justify left))
     )
-    (property "Value" "10k" (id 1) (at 253.238 108.3822 0)
+    (property "Value" "1meg" (id 1) (at 253.238 108.3822 0)
       (effects (font (size 1.27 1.27)) (justify left))
     )
@@
     (pin "2")
   )
-  (symbol (lib_id "Connector:TestPoint") (at 227.33 99.06 0) (unit 1)
-    (in_bom yes) (on_board yes) (fields_autoplaced)
-    (property "Reference" "TP12" (id 0) (at 228.727 94.9233 0)
-      (effects (font (size 1.27 1.27)) (justify left))
-    )
-    (property "Value" "TestPoint" (id 1) (at 228.727 97.4602 0)
-      (effects (font (size 1.27 1.27)) (justify left))
-    )
-    (property "Footprint" "Connector_Pin:Pin_D0.7mm_L6.5mm_W1.8mm_FlatFork" (id 2) (at 232.41 99.06 0)
-      (effects (font (size 1.27 1.27)) hide)
-    )
-    (property "Datasheet" "~" (id 3) (at 232.41 99.06 0)
-      (effects (font (size 1.27 1.27)) hide)
-    )
-    (pin "1")
-  )
   (symbol (lib_id "degson:DG3XX-02-5.0") (at 107.95 34.29 270) (unit 1)
     (in_bom yes) (on_board yes) (fields_autoplaced)
@@
     )
     (path "/7ffe756e-7031-40a9-a22e-c934089443a6"
-      (reference "R9") (unit 1) (value "10k") (footprint "Resistor_SMD:R_0805_2012Metric_Pad1.20x1.40mm_HandSolder")
+      (reference "R9") (unit 1) (value "1meg") (footprint "Resistor_SMD:R_0805_2012Metric_Pad1.20x1.40mm_HandSolder")
     )
     (path "/0e9de456-4848-46ec-9fa8-1e86ac24055c"
@@
       (reference "TP11") (unit 1) (value "TestPoint") (footprint "Connector_Pin:Pin_D0.7mm_L6.5mm_W1.8mm_FlatFork")
     )
-    (path "/f181baca-340c-4570-b197-b9647a3ba278"
-      (reference "TP12") (unit 1) (value "TestPoint") (footprint "Connector_Pin:Pin_D0.7mm_L6.5mm_W1.8mm_FlatFork")
-    )
     (path "/cab9d3f3-ba3f-4024-b3d6-87696cb91a7a"
